File: hardware/controlPanel/controlPanel.kicad_pcb (KiCad board)
At the start: 2 copper layers, 30.2 x 35.2 mm, 20 parts, among them J1 Power Supply, J2 Conn_01x08_Female, SW1 Ein/Aus, SW2 Fallschirm schließen, U1 LM555xM

Commit message: changed the footprint of the connector to the controlPanel and changed the order of the pin numbers
Parts:
- moved J2 14.0 mm to (165.9, 83.8), turned to 180 degrees
Connections:
- J2 pad 1: +12V -> Net-(J2-Pad1)
- J2 pad 2: /Batt+ -> Net-(J2-Pad2)
- J2 pad 3: /Network_LED -> /Boot_LED
- J2 pad 4: GND -> /GPS_LED
- J2 pad 5: /GPS_LED -> GND
- J2 pad 6: /Boot_LED -> /Network_LED
- J2 pad 7: Net-(J2-Pad7) -> /Batt+
- J2 pad 8: Net-(J2-Pad8) -> +12V
- R6 pad 1: Net-(J2-Pad7) -> Net-(J2-Pad2)
- R6 pad 2: Net-(J2-Pad8) -> Net-(J2-Pad1)
- SW2 pad 2: Net-(J2-Pad8) -> Net-(J2-Pad1)
Routing:
- net Net-(J2-Pad1): track 0.00 -> 13.8 mm
- net Net-(J2-Pad8): track 13.8 -> 0.00 mm
- net Net-(J2-Pad7): track 3.04 -> 0.00 mm
- net Net-(J2-Pad2): track 0.00 -> 3.03 mm
