File: hardware/powerBoard/powerBoard.kicad_sch (KiCad schematic)
At the start: 25 parts, among them J1 Batt, J2 Berry IMU, J3 Control_Panel, J4 Servo_1, J5 Servo_2, J6 Servo_3, J7 Raspi, J8 Masse, U1 R-78C5.0-1.0, U2 DRV8801PWP

Commit message: changed the footprint of the connector to the controlPanel and changed the order of the pin numbers
Parts:
- J3: footprint Connector_PinHeader_2.54mm:PinHeader_2x04_P2.54mm_Vertical -> Connector_IDC:IDC-Header_2x04_P2.54mm_Vertical
Connections:
- net +12V: now also J3.8 (Pin_8); no longer J3.1 (Pin_1)
- net +5V: now also J3.2 (Pin_2); no longer J3.7 (Pin_7)
- net BOOT-LED: now also J3.3 (Pin_3); no longer J3.6 (Pin_6)
- net Batt+: now also J3.7 (Pin_7); no longer J3.2 (Pin_2)
- net Button-Pin: now also J3.1 (Pin_1); no longer J3.8 (Pin_8)
- net GND: now also J3.5 (Pin_5); no longer J3.4 (Pin_4)
- net GPS-LED: now also J3.4 (Pin_4); no longer J3.5 (Pin_5)
- net Network-LED: now also J3.6 (Pin_6); no longer J3.3 (Pin_3)
Other:
- moved on the sheet: J3
Changed lines of the file:
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@@
     (pin "1")
   )
-  (symbol (lib_id "Connector_Generic:Conn_02x04_Top_Bottom") (at 59.69 143.51 0) (unit 1)
+  (symbol (lib_id "Connector_Generic:Conn_02x04_Top_Bottom") (at 62.23 146.05 180) (unit 1)
     (in_bom yes) (on_board yes) (fields_autoplaced)
     (property "Reference" "J3" (id 0) (at 60.96 134.62 0))
     (property "Value" "Control_Panel" (id 1) (at 60.96 137.16 0))
-    (property "Footprint" "Connector_PinHeader_2.54mm:PinHeader_2x04_P2.54mm_Vertical" (id 2) (at 59.69 143.51 0)
-      (effects (font (size 1.27 1.27)) hide)
-    )
-    (property "Datasheet" "~" (id 3) (at 59.69 143.51 0)
+    (property "Footprint" "Connector_IDC:IDC-Header_2x04_P2.54mm_Vertical" (id 2) (at 62.23 146.05 0)
+      (effects (font (size 1.27 1.27)) hide)
+    )
+    (property "Datasheet" "~" (id 3) (at 62.23 146.05 0)
       (effects (font (size 1.27 1.27)) hide)
     )
@@
     )
     (path "/ab51f4e7-2bf8-422b-b09b-1a8a5c45ad1d"
-      (reference "J3") (unit 1) (value "Control_Panel") (footprint "Connector_PinHeader_2.54mm:PinHeader_2x04_P2.54mm_Vertical")
+      (reference "J3") (unit 1) (value "Control_Panel") (footprint "Connector_IDC:IDC-Header_2x04_P2.54mm_Vertical")
     )
     (path "/a3bc0c62-09a8-4287-b969-1d6c77f476ed"
